File: ClockModule/ClockModule.kicad_sch (KiCad schematic)
At the start: 1 part, among them J1 Conn_01x05_Pin

Commit message: Final clock updates
Parts:
- J1: footprint Connector_PinHeader_1.00mm:PinHeader_1x05_P1.00mm_Horizontal -> Connector_PinHeader_2.54mm:PinHeader_1x05_P2.54mm_Vertical
Connections:
- net +5V: now also J1.1 (Pin_1); no longer J1.2 (Pin_2)
- net GND: now also J1.2 (Pin_2); no longer J1.1 (Pin_1)
Changed lines of the file:
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@@
 	(paper "A4")
+	(junction
+		(at 168.91 50.8)
+		(diameter 0)
+		(color 0 0 0 0)
+	)
 	(junction
 		(at 168.91 48.26)
@@
 		(color 0 0 0 0)
 	)
-	(junction
-		(at 168.91 50.8)
-		(diameter 0)
-		(color 0 0 0 0)
-	)
 	(wire
 		(pts
@@
 	(wire
 		(pts
-			(xy 165.1 50.8) (xy 168.91 50.8)
-		)
-		(stroke
-			(width 0)
-			(type default)
-		)
-	)
-	(wire
-		(pts
 			(xy 71.12 44.45) (xy 54.61 44.45)
 		)
@@
 	(wire
 		(pts
-			(xy 165.1 52.07) (xy 165.1 50.8)
-		)
-		(stroke
-			(width 0)
-			(type default)
-		)
-	)
-	(wire
-		(pts
 			(xy 172.72 45.72) (xy 179.07 45.72)
 		)
@@
 	(wire
 		(pts
+			(xy 168.91 48.26) (xy 179.07 48.26)
+		)
+		(stroke
+			(width 0)
+			(type default)
+		)
+	)
+	(wire
+		(pts
 			(xy 168.91 46.99) (xy 168.91 48.26)
 		)
@@
 	(wire
 		(pts
-			(xy 168.91 48.26) (xy 179.07 48.26)
+			(xy 166.37 50.8) (xy 168.91 50.8)
 		)
 		(stroke
@@
 	(wire
 		(pts
-			(xy 165.1 46.99) (xy 165.1 48.26)
-		)
-		(stroke
-			(width 0)
-			(type default)
-		)
-	)
-	(wire
-		(pts
 			(xy 102.87 41.91) (xy 105.41 41.91)
 		)
@@
 	(wire
 		(pts
-			(xy 165.1 48.26) (xy 168.91 48.26)
+			(xy 166.37 46.99) (xy 166.37 48.26)
+		)
+		(stroke
+			(width 0)
+			(type default)
+		)
+	)
+	(wire
+		(pts
+			(xy 166.37 48.26) (xy 168.91 48.26)
 		)
 		(stroke
@@
 		(pts
 			(xy 172.72 40.64) (xy 179.07 40.64)
+		)
+		(stroke
+			(width 0)
+			(type default)
+		)
+	)
+	(wire
+		(pts
+			(xy 166.37 52.07) (xy 166.37 50.8)
 		)
 		(stroke
@@
 	(symbol
 		(lib_id "power:+5V")
-		(at 165.1 46.99 0)
+		(at 166.37 52.07 180)
 		(unit 1)
 		(exclude_from_sim no)
@@
 		(fields_autoplaced yes)
 		(property "Reference" "#PWR01"
-			(at 165.1 50.8 0)
+			(at 166.37 48.26 0)
 			(effects
 				(font
@@
 		)
 		(property "Value" "+5V"
-			(at 165.1 41.91 0)
+			(at 166.37 57.15 0)
 			(effects
 				(font
@@
 		)
 		(property "Footprint" ""
-			(at 165.1 46.99 0)
+			(at 166.37 52.07 0)
 			(effects
 				(font
@@
 		)
 		(property "Datasheet" ""
-			(at 165.1 46.99 0)
+			(at 166.37 52.07 0)
 			(effects
 				(font
@@
 		)
 		(property "Description" "Power symbol creates a global label with name \"+5V\""
-			(at 165.1 46.99 0)
+			(at 166.37 52.07 0)
 			(effects
 				(font
@@
 	(symbol
 		(lib_id "power:GND")
-		(at 165.1 52.07 0)
+		(at 166.37 46.99 180)
 		(unit 1)
 		(exclude_from_sim no)
@@
 		(fields_autoplaced yes)
 		(property "Reference" "#PWR02"
-			(at 165.1 58.42 0)
+			(at 166.37 40.64 0)
 			(effects
 				(font
@@
 		)
 		(property "Value" "GND"
-			(at 165.1 57.15 0)
+			(at 166.37 41.91 0)
 			(effects
 				(font
@@
 		)
 		(property "Footprint" ""
-			(at 165.1 52.07 0)
+			(at 166.37 46.99 0)
 			(effects
 				(font
@@
 		)
 		(property "Datasheet" ""
-			(at 165.1 52.07 0)
+			(at 166.37 46.99 0)
 			(effects
 				(font
@@
 		)
 		(property "Description" "Power symbol creates a global label with name \"GND\" , ground"
-			(at 165.1 52.07 0)
+			(at 166.37 46.99 0)
 			(effects
 				(font
@@
 			)
 		)
-		(property "Footprint" "Connector_PinHeader_1.00mm:PinHeader_1x05_P1.00mm_Horizontal"
+		(property "Footprint" "Connector_PinHeader_2.54mm:PinHeader_1x05_P2.54mm_Vertical"
 			(at 184.15 45.72 0)
 			(effects
