File: ClockModule/astable_clock.kicad_sch (KiCad schematic)
At the start: 9 parts, among them U7 LM555xN

Commit message: Final clock updates
Parts:
- D1: renamed from D4; footprint LED_THT:LED_D2.0mm_W4.8mm_H2.5mm_FlatTop -> LED_THT:LED_D5.0mm
- renumbered C9 to C1, C10 to C2, R10 to R1, RV2 to RV1, U7 to U1
Changed lines of the file:
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@@
 		(on_board yes)
 		(dnp no)
-		(property "Reference" "U7"
+		(property "Reference" "U1"
 			(at 139.7 87.884 0)
 			(effects
@@
 		(pin "4"
 		)
-		(instances)
+		(instances
+			(project ""
+				(path "/54ad16a3-0854-4bc5-acd6-428be9af167c/8cdd56ee-c324-45fe-a470-757d2dbc6b80"
+					(reference "U1")
+					(unit 1)
+				)
+			)
+		)
 	)
 	(symbol
@@
 		(dnp no)
 		(fields_autoplaced yes)
-		(property "Reference" "D4"
+		(property "Reference" "D1"
 			(at 191.77 96.8374 90)
 			(effects
@@
 			)
 		)
-		(property "Footprint" "LED_THT:LED_D2.0mm_W4.8mm_H2.5mm_FlatTop"
+		(property "Footprint" "LED_THT:LED_D5.0mm"
 			(at 187.96 96.52 0)
 			(effects
@@
 		(pin "2"
 		)
-		(instances)
+		(instances
+			(project ""
+				(path "/54ad16a3-0854-4bc5-acd6-428be9af167c/8cdd56ee-c324-45fe-a470-757d2dbc6b80"
+					(reference "D1")
+					(unit 1)
+				)
+			)
+		)
 	)
 	(symbol
@@
 		(dnp no)
 		(fields_autoplaced yes)
-		(property "Reference" "R10"
+		(property "Reference" "R1"
 			(at 166.37 81.2799 0)
 			(effects
@@
 		(pin "2"
 		)
-		(instances)
+		(instances
+			(project ""
+				(path "/54ad16a3-0854-4bc5-acd6-428be9af167c/8cdd56ee-c324-45fe-a470-757d2dbc6b80"
+					(reference "R1")
+					(unit 1)
+				)
+			)
+		)
 	)
 	(symbol
@@
 		(dnp no)
 		(fields_autoplaced yes)
-		(property "Reference" "C10"
+		(property "Reference" "C2"
 			(at 138.43 110.8709 0)
 			(effects
@@
 		(pin "2"
 		)
-		(instances)
+		(instances
+			(project ""
+				(path "/54ad16a3-0854-4bc5-acd6-428be9af167c/8cdd56ee-c324-45fe-a470-757d2dbc6b80"
+					(reference "C2")
+					(unit 1)
+				)
+			)
+		)
 	)
 	(symbol
@@
 		(dnp no)
 		(fields_autoplaced yes)
-		(property "Reference" "C9"
+		(property "Reference" "C1"
 			(at 124.46 111.7599 0)
 			(effects
@@
 		(pin "1"
 		)
-		(instances)
+		(instances
+			(project ""
+				(path "/54ad16a3-0854-4bc5-acd6-428be9af167c/8cdd56ee-c324-45fe-a470-757d2dbc6b80"
+					(reference "C1")
+					(unit 1)
+				)
+			)
+		)
 	)
 	(symbol
@@
 		(dnp no)
 		(fields_autoplaced yes)
-		(property "Reference" "#PWR020"
+		(property "Reference" "#PWR04"
 			(at 148.59 125.73 0)
 			(effects
@@
 		(dnp no)
 		(fields_autoplaced yes)
-		(property "Reference" "RV2"
+		(property "Reference" "RV1"
 			(at 180.34 95.2499 0)
 			(effects
@@
 		(pin "2"
 		)
-		(instances)
+		(instances
+			(project ""
+				(path "/54ad16a3-0854-4bc5-acd6-428be9af167c/8cdd56ee-c324-45fe-a470-757d2dbc6b80"
+					(reference "RV1")
+					(unit 1)
+				)
+			)
+		)
 	)
 	(symbol
@@
 		(dnp no)
 		(fields_autoplaced yes)
-		(property "Reference" "#PWR019"
+		(property "Reference" "#PWR03"
 			(at 148.59 72.39 0)
 			(effects
