File: ClockModule/clock_select.kicad_sch (KiCad schematic)
At the start: 5 parts, among them U3 OR, U4 NOT

Commit message: Final clock updates
Parts:
- D3: footprint LED_THT:LED_D2.0mm_W4.8mm_H2.5mm_FlatTop -> LED_THT:LED_D5.0mm
Changed lines of the file:
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@@
 			)
 		)
-		(property "Footprint" "LED_THT:LED_D2.0mm_W4.8mm_H2.5mm_FlatTop"
+		(property "Footprint" "LED_THT:LED_D5.0mm"
 			(at 147.32 100.33 0)
 			(effects
