File: ClockModule/bistable_debouncing_circuit.kicad_sch (KiCad schematic)
At the start: 6 parts, among them SW1 SW_SPDT, U6 LM555xN

Commit message: Switch pull up resistor was connected to wrong pin. Connected to switch now
Connections:
- net at SW1.3 (C), U6.4 (R): now also R9.1
- net at C7.1, U6.5 (CV): no longer R9.1
Changed lines of the file:
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@@
 	(paper "A4")
 	(junction
+		(at 92.71 87.63)
+		(diameter 0)
+		(color 0 0 0 0)
+	)
+	(junction
 		(at 92.71 55.88)
 		(diameter 0)
@@
 	(junction
 		(at 85.09 77.47)
-		(diameter 0)
-		(color 0 0 0 0)
-	)
-	(junction
-		(at 92.71 82.55)
 		(diameter 0)
 		(color 0 0 0 0)
@@
 	(wire
 		(pts
-			(xy 83.82 87.63) (xy 95.25 87.63)
-		)
-		(stroke
-			(width 0)
-			(type default)
-		)
-	)
-	(wire
-		(pts
-			(xy 92.71 82.55) (xy 95.25 82.55)
+			(xy 83.82 87.63) (xy 92.71 87.63)
+		)
+		(stroke
+			(width 0)
+			(type default)
+		)
+	)
+	(wire
+		(pts
+			(xy 88.9 82.55) (xy 95.25 82.55)
 		)
 		(stroke
@@
 	(wire
 		(pts
-			(xy 88.9 82.55) (xy 92.71 82.55)
-		)
-		(stroke
-			(width 0)
-			(type default)
-		)
-	)
-	(wire
-		(pts
 			(xy 88.9 104.14) (xy 107.95 104.14)
 		)
@@
 	(wire
 		(pts
+			(xy 92.71 87.63) (xy 95.25 87.63)
+		)
+		(stroke
+			(width 0)
+			(type default)
+		)
+	)
+	(wire
+		(pts
 			(xy 72.39 85.09) (xy 72.39 104.14)
 		)
@@
 	(wire
 		(pts
+			(xy 111.76 57.15) (xy 111.76 55.88)
+		)
+		(stroke
+			(width 0)
+			(type default)
+		)
+	)
+	(wire
+		(pts
+			(xy 120.65 87.63) (xy 121.92 87.63)
+		)
+		(stroke
+			(width 0)
+			(type default)
+		)
+	)
+	(wire
+		(pts
 			(xy 85.09 77.47) (xy 95.25 77.47)
 		)
@@
 	(wire
 		(pts
-			(xy 111.76 57.15) (xy 111.76 55.88)
-		)
-		(stroke
-			(width 0)
-			(type default)
-		)
-	)
-	(wire
-		(pts
-			(xy 120.65 87.63) (xy 121.92 87.63)
-		)
-		(stroke
-			(width 0)
-			(type default)
-		)
-	)
-	(wire
-		(pts
 			(xy 85.09 64.77) (xy 85.09 55.88)
 		)
@@
 	(wire
 		(pts
+			(xy 92.71 72.39) (xy 92.71 87.63)
+		)
+		(stroke
+			(width 0)
+			(type default)
+		)
+	)
+	(wire
+		(pts
 			(xy 85.09 55.88) (xy 92.71 55.88)
 		)
 		(stroke
-			(width 0)
-			(type default)
-		)
-	)
-	(wire
-		(pts
-			(xy 92.71 72.39) (xy 92.71 82.55)
-		)
-		(stroke
