File: MemoryAccessRegister/MemoryAccessRegister.kicad_sch (KiCad schematic)
At the start: 16 parts, among them J1 Conn_01x04_Pin, J2 Conn_01x04_Pin, J3 Conn_01x06_Pin, SW1 SW_SPDT, U1 CD74HCT258E, U3 74LS173

Commit message: Fixed LED and pin footprints for MAR and cleaned up the layout
Parts:
- removed J1, J2: Conn_01x04_Pin, Connector_PinHeader_1.00mm:PinHeader_1x04_P1.00mm_Horizontal, symbol Connector:Conn_01x04_Pin
- added J4: Conn_01x05_Pin, Connector_PinHeader_2.54mm:PinHeader_1x05_P2.54mm_Vertical, symbol Connector:Conn_01x05_Pin
- added J5: Conn_01x03_Pin, Connector_PinHeader_2.54mm:PinHeader_1x03_P2.54mm_Vertical, symbol Connector:Conn_01x03_Pin
- D1, D2: footprint LED_THT:LED_D2.0mm_W4.8mm_H2.5mm_FlatTop -> LED_THT:LED_D5.0mm
- D3: renamed from D4; footprint LED_THT:LED_D2.0mm_W4.8mm_H2.5mm_FlatTop -> LED_THT:LED_D5.0mm
- D4: renamed from D6; footprint LED_THT:LED_D2.0mm_W4.8mm_H2.5mm_FlatTop -> LED_THT:LED_D5.0mm
- J2: renamed from J3; footprint Connector_PinHeader_1.00mm:PinHeader_1x06_P1.00mm_Horizontal -> Connector_PinHeader_2.54mm:PinHeader_1x06_P2.54mm_Vertical
- renumbered R4 to R3, R6 to R4
Connections:
- net +5V: now also J2.1 (Pin_1); no longer J2.6 (Pin_6)
- net A0: now also J4.2 (Pin_2)
- net A1: now also J4.3 (Pin_3)
- net A2: now also J4.4 (Pin_4)
- net A3: now also J4.5 (Pin_5)
- net Bus 0: now also J2.3 (Pin_3)
- net Bus 1: now also J2.4 (Pin_4)
- net Bus 2: now also J2.5 (Pin_5)
- net Bus 3: now also J2.6 (Pin_6)
- net CLK: now also J5.3 (Pin_3); no longer J2.3 (Pin_3)
- net GND: now also J2.2 (Pin_2); no longer J2.5 (Pin_5)
- net Program: now also J4.1 (Pin_1); no longer J2.4 (Pin_4)
- net RST: now also J5.2 (Pin_2); no longer J2.2 (Pin_2)
- net ~En: now also J5.1 (Pin_1); no longer J2.1 (Pin_1)
Other:
- moved on the sheet: J2
