File: MemoryAccessRegister/MemoryAccessRegister.kicad_pcb (KiCad board)
At the start: 2 copper layers, 84.3 x 39.2 mm, 26 parts, among them J1 Conn_01x05_Pin, J2 Conn_01x06_Pin, J3 Conn_01x03_Pin, SW1 SW_SPDT, U1 SN74AC14N, U2 CD74HCT258E, U4 74LS173

Commit message: Manufacturer footprint and data sheet seem to be wrong for the mux. Input for bits 3 and 4 are swapped.
Connections:
- U2 pad 10: /Prog 3 -> /B3
- U2 pad 11: /B3 -> /Prog 3
- U2 pad 13: /Prog 2 -> /B2
- U2 pad 14: /B2 -> /Prog 2
Routing:
- net /B3: track 25.4 -> 22.8 mm
- net /Prog 2: track 48.4 -> 50.9 mm
- net /B2: track 30.4 -> 27.9 mm
- net /Prog 3: track 38.5 -> 39.6 mm
Changed lines of the file:
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@@
 			(layers "*.Cu" "*.Mask")
 			(remove_unused_layers no)
-			(net 19 "/Prog 3")
-			(pinfunction "3A")
+			(net 20 "/B3")
+			(pinfunction "3B")
 			(pintype "input")
 		)
@@
 			(layers "*.Cu" "*.Mask")
 			(remove_unused_layers no)
-			(net 20 "/B3")
-			(pinfunction "3B")
+			(net 19 "/Prog 3")
+			(pinfunction "3A")
 			(pintype "input")
 		)
@@
 			(layers "*.Cu" "*.Mask")
 			(remove_unused_layers no)
-			(net 25 "/Prog 2")
-			(pinfunction "4A")
+			(net 21 "/B2")
+			(pinfunction "4B")
 			(pintype "input")
 		)
@@
 			(layers "*.Cu" "*.Mask")
 			(remove_unused_layers no)
-			(net 21 "/B2")
-			(pinfunction "4B")
+			(net 25 "/Prog 2")
+			(pinfunction "4A")
 			(pintype "input")
 		)
@@
 	)
 	(segment
-		(start 198.5 80.1)
-		(end 204.4 86)
+		(start 195.96 77.56)
+		(end 195.96 77.25)
 		(width 0.2)
 		(layer "B.Cu")
@@
 	)
 	(segment
-		(start 198.5 77.25)
-		(end 198.5 80.1)
+		(start 212.96 86)
+		(end 204.4 86)
 		(width 0.2)
 		(layer "B.Cu")
@@
 	)
 	(segment
-		(start 212.96 86)
-		(end 215.46 88.5)
+		(start 204.4 86)
+		(end 195.96 77.56)
 		(width 0.2)
 		(layer "B.Cu")
@@
 	)
 	(segment
-		(start 204.4 86)
+		(start 215.46 88.5)
 		(end 212.96 86)
 		(width 0.2)
@@
 	)
 	(segment
-		(start 201.28 82.57)
-		(end 195.96 77.25)
+		(start 218.17 84.87)
+		(end 213.3 80)
 		(width 0.2)
 		(layer "F.Cu")
@@
 	)
 	(segment
-		(start 218.17 84.87)
-		(end 215.87 82.57)
+		(start 213.3 80)
+		(end 201.25 80)
 		(width 0.2)
 		(layer "F.Cu")
@@
 	)
 	(segment
-		(start 215.87 82.57)
-		(end 201.28 82.57)
+		(start 201.25 80)
+		(end 198.5 77.25)
 		(width 0.2)
 		(layer "F.Cu")
@@
 	)
 	(segment
-		(start 215.63 84.87)
-		(end 215.064315 84.87)
+		(start 194.03 80.4)
+		(end 190.88 77.25)
 		(width 0.2)
 		(layer "F.Cu")
@@
 	)
 	(segment
-		(start 215.064315 84.87)
-		(end 213.164315 82.97)
+		(start 215.63 84.87)
+		(end 215.064315 84.87)
 		(width 0.2)
 		(layer "F.Cu")
@@
 	)
 	(segment
-		(start 194.06 82.97)
-		(end 188.34 77.25)
+		(start 210.594315 80.4)
+		(end 194.03 80.4)
 		(width 0.2)
 		(layer "F.Cu")
@@
 	)
 	(segment
-		(start 213.164315 82.97)
-		(end 194.06 82.97)
+		(start 215.064315 84.87)
+		(end 210.594315 80.4)
 		(width 0.2)
 		(layer "F.Cu")
@@
 	)
 	(segment
-		(start 212.794314 86.4)
-		(end 214.36 87.965686)
+		(start 216.9 89.6)
+		(end 215.004365 89.6)
 		(width 0.2)
 		(layer "B.Cu")
@@
 	)
 	(segment
-		(start 214.36 87.965686)
-		(end 214.36 88.955635)
+		(start 214.36 88.955635)
+		(end 214.36 87.965686)
 		(width 0.2)
 		(layer "B.Cu")
@@
 	)
 	(segment
-		(start 196.032014 78.1977)
+		(start 212.794314 86.4)
 		(end 204.234314 86.4)
 		(width 0.2)
@@
 	)
 	(segment
-		(start 216.9 89.6)
-		(end 218 88.5)
+		(start 189.2877 78.1977)
+		(end 188.34 77.25)
 		(width 0.2)
 		(layer "B.Cu")
@@
 	(segment
 		(start 204.234314 86.4)
-		(end 212.794314 86.4)
+		(end 196.032014 78.1977)
 		(width 0.2)
 		(layer "B.Cu")
@@
 	)
 	(segment
-		(start 214.36 88.955635)
-		(end 215.004365 89.6)
+		(start 214.36 87.965686)
+		(end 212.794314 86.4)
 		(width 0.2)
 		(layer "B.Cu")
@@
 	)
 	(segment
-		(start 191.8277 78.1977)
-		(end 196.032014 78.1977)
+		(start 215.004365 89.6)
+		(end 214.36 88.955635)
 		(width 0.2)
 		(layer "B.Cu")
@@
 	)
 	(segment
-		(start 190.88 77.25)
-		(end 191.8277 78.1977)
+		(start 218 88.5)
+		(end 216.9 89.6)
 		(width 0.2)
 		(layer "B.Cu")
@@
 	)
 	(segment
-		(start 215.004365 89.6)
-		(end 216.9 89.6)
+		(start 196.032014 78.1977)
+		(end 189.2877 78.1977)
 		(width 0.2)
 		(layer "B.Cu")
