File: Bus/bus.kicad_pcb (KiCad board)
At the start: 2 copper layers, 0 parts

Commit message: Some initial bus layout
Parts:
- added D1: LED, LED_THT:LED_D5.0mm, F.Cu at (148.1, 21.1)
- added D2: LED, LED_THT:LED_D5.0mm, F.Cu at (141.5, 21.1)
- added D3: LED, LED_THT:LED_D5.0mm, F.Cu at (134.9, 21.1)
- added D4: LED, LED_THT:LED_D5.0mm, F.Cu at (128.3, 21.1)
- added D5: LED, LED_THT:LED_D5.0mm, F.Cu at (121.7, 21.1)
- added D6: LED, LED_THT:LED_D5.0mm, F.Cu at (115.1, 21.1)
- added D7: LED, LED_THT:LED_D5.0mm, F.Cu at (108.5, 21.1)
- added D8: LED, LED_THT:LED_D5.0mm, F.Cu at (101.9, 21.1)
- added J1: Conn_01x05_Pin, Connector_PinHeader_2.54mm:PinHeader_1x05_P2.54mm_Vertical, F.Cu at (104.5, 41.4)
- added J10: USB_C_Receptacle_PowerOnly_6P, Connector_USB:USB_C_Receptacle_GCT_USB4085, F.Cu at (122.1, 184.2)
- added J11: Conn_01x10_Pin, Connector_PinHeader_2.54mm:PinHeader_1x10_P2.54mm_Vertical, F.Cu at (156.0, 33.5)
- added J12: Conn_01x05_Pin, Connector_PinHeader_2.54mm:PinHeader_1x05_P2.54mm_Vertical, F.Cu at (151.9, 34.8)
- added J2: Conn_01x08_Pin, Connector_PinHeader_2.54mm:PinHeader_1x08_P2.54mm_Vertical, F.Cu at (155.8, 62.0)
- added J3: Conn_01x06_Pin, Connector_PinHeader_2.54mm:PinHeader_1x06_P2.54mm_Vertical, F.Cu at (152.1, 60.7)
- added J4: Conn_01x08_Pin, Connector_PinHeader_2.54mm:PinHeader_1x08_P2.54mm_Vertical, F.Cu at (156.0, 112.0)
- added J5: Conn_01x06_Pin, Connector_PinHeader_2.54mm:PinHeader_1x06_P2.54mm_Vertical, F.Cu at (151.9, 110.7)
- added J6: Conn_01x08_Pin, Connector_PinHeader_2.54mm:PinHeader_1x08_P2.54mm_Vertical, F.Cu at (103.8, 62.0)
- added J7: Conn_01x06_Pin, Connector_PinHeader_2.54mm:PinHeader_1x06_P2.54mm_Vertical, F.Cu at (108.0, 63.2)
- added J8: Conn_01x10_Pin, Connector_PinHeader_2.54mm:PinHeader_1x10_P2.54mm_Vertical, F.Cu at (155.7, 83.6)
- added J9: Conn_01x06_Pin, Connector_PinHeader_2.54mm:PinHeader_1x06_P2.54mm_Vertical, F.Cu at (151.9, 84.8)
- added R1: 10k, _DownloadFootprints:CF_series_Resistors_THT, F.Cu at (113.5, 163.1)
- added R10: 220, _DownloadFootprints:CF_series_Resistors_THT, F.Cu at (141.5, 18.1)
- added R11: 220, _DownloadFootprints:CF_series_Resistors_THT, F.Cu at (134.9, 18.1)
- added R12: 220, _DownloadFootprints:CF_series_Resistors_THT, F.Cu at (128.3, 18.1)
- added R13: 220, _DownloadFootprints:CF_series_Resistors_THT, F.Cu at (121.7, 18.1)
- added R14: 220, _DownloadFootprints:CF_series_Resistors_THT, F.Cu at (115.1, 18.1)
- added R15: 220, _DownloadFootprints:CF_series_Resistors_THT, F.Cu at (108.5, 18.1)
- added R16: 220, _DownloadFootprints:CF_series_Resistors_THT, F.Cu at (101.9, 18.1)
- added R17: 5.1k, _DownloadFootprints:CF_series_Resistors_THT, F.Cu at (116.8, 176.8)
- added R18: 5.1k, _DownloadFootprints:CF_series_Resistors_THT, F.Cu at (133.3, 188.2)
- added R2: 10k, _DownloadFootprints:CF_series_Resistors_THT, F.Cu at (116.8, 163.1)
- added R3: 10k, _DownloadFootprints:CF_series_Resistors_THT, F.Cu at (120.1, 163.1)
- added R4: 10k, _DownloadFootprints:CF_series_Resistors_THT, F.Cu at (123.4, 163.1)
- added R5: 10k, _DownloadFootprints:CF_series_Resistors_THT, F.Cu at (126.7, 163.1)
- added R6: 10k, _DownloadFootprints:CF_series_Resistors_THT, F.Cu at (130.0, 163.1)
- added R7: 10k, _DownloadFootprints:CF_series_Resistors_THT, F.Cu at (133.3, 163.1)
- added R8: 10k, _DownloadFootprints:CF_series_Resistors_THT, F.Cu at (136.7, 163.1)
- added R9: 220, _DownloadFootprints:CF_series_Resistors_THT, F.Cu at (148.1, 18.1)
Routing:
- net /B7: track 0.00 -> 310.7 mm, vias 0 -> 4
- net /B6: track 0.00 -> 299.7 mm, vias 0 -> 4
- net /B5: track 0.00 -> 293.3 mm, vias 0 -> 4
- net /B4: track 0.00 -> 287.6 mm, vias 0 -> 4
- net /B3: track 0.00 -> 262.5 mm, vias 0 -> 4
- net /B2: track 0.00 -> 261.8 mm, vias 0 -> 4
- net /B1: track 0.00 -> 261.6 mm, vias 0 -> 4
- net /B0: track 0.00 -> 260.4 mm, vias 0 -> 4
- net /CLK: track 0.00 -> 240.8 mm, vias 0 -> 6
- net /~RST: track 0.00 -> 160.5 mm, vias 0 -> 2
- net /RST: track 0.00 -> 142.3 mm, vias 0 -> 3
- net /PC ~CO: track 0.00 -> 107.8 mm
- net /PC CE: track 0.00 -> 99.9 mm
- net /PC ~JMP: track 0.00 -> 97.1 mm
- net /~CLK: track 0.00 -> 91.0 mm, vias 0 -> 1
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- added copper zone on In1.Cu, net +5V
- added copper zone on In2.Cu, net GND
Other:
- board outline added: 69.3 x 213.7 mm
- copper layers 2 -> 4
