File: Bus/ram.kicad_sch (KiCad schematic)
At the start: 2 parts, among them J20 Conn_01x03_Pin, J21 Conn_01x10_Pin

Commit message: Updated bus schmatic pins to match final layouts
Parts:
- renumbered J21 to J17, J20 to J18
Connections:
- net ~{WO} renamed ~{RO}
Other:
- moved on the sheet: J18
Changed lines of the file:
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@@
 	(hierarchical_label "RI"
 		(shape input)
-		(at 99.06 97.79 180)
+		(at 100.33 147.32 180)
 		(fields_autoplaced yes)
 		(effects
@@
 	(hierarchical_label "CLK"
 		(shape input)
-		(at 99.06 100.33 180)
+		(at 100.33 144.78 180)
 		(fields_autoplaced yes)
 		(effects
@@
 		)
 	)
-	(hierarchical_label "~{WO}"
+	(hierarchical_label "~{RO}"
 		(shape input)
-		(at 99.06 102.87 180)
+		(at 100.33 142.24 180)
 		(fields_autoplaced yes)
 		(effects
@@
 		(dnp no)
 		(fields_autoplaced yes)
-		(property "Reference" "#PWR025"
+		(property "Reference" "#PWR020"
 			(at 92.71 118.11 0)
 			(effects
@@
 			(project "bus"
 				(path "/37ae8b13-e183-404e-b70a-681e1af60f55/61b8f38e-6730-4fc5-8ab9-627730f56fd6"
-					(reference "#PWR025")
+					(reference "#PWR020")
 					(unit 1)
 				)
@@
 		(dnp no)
 		(fields_autoplaced yes)
-		(property "Reference" "J21"
+		(property "Reference" "J17"
 			(at 106.68 125.7299 0)
 			(effects
@@
 			(project "bus"
 				(path "/37ae8b13-e183-404e-b70a-681e1af60f55/61b8f38e-6730-4fc5-8ab9-627730f56fd6"
-					(reference "J21")
+					(reference "J17")
 					(unit 1)
 				)
@@
 	(symbol
 		(lib_id "Connector:Conn_01x03_Pin")
-		(at 104.14 100.33 180)
+		(at 105.41 144.78 0)
+		(mirror y)
 		(unit 1)
 		(exclude_from_sim no)
@@
 		(dnp no)
 		(fields_autoplaced yes)
-		(property "Reference" "J20"
-			(at 105.41 99.0599 0)
+		(property "Reference" "J18"
+			(at 106.68 146.0501 0)
 			(effects
 				(font
@@
 		)
 		(property "Value" "Conn_01x03_Pin"
-			(at 105.41 101.5999 0)
+			(at 106.68 143.5101 0)
 			(effects
 				(font
@@
 		)
 		(property "Footprint" "Connector_PinHeader_2.54mm:PinHeader_1x03_P2.54mm_Vertical"
-			(at 104.14 100.33 0)
+			(at 105.41 144.78 0)
 			(effects
 				(font
@@
 		)
 		(property "Datasheet" "~"
-			(at 104.14 100.33 0)
+			(at 105.41 144.78 0)
 			(effects
 				(font
@@
 		)
 		(property "Description" "Generic connector, single row, 01x03, script generated"
-			(at 104.14 100.33 0)
+			(at 105.41 144.78 0)
 			(effects
 				(font
@@
 			(project "bus"
 				(path "/37ae8b13-e183-404e-b70a-681e1af60f55/61b8f38e-6730-4fc5-8ab9-627730f56fd6"
-					(reference "J20")
+					(reference "J18")
 					(unit 1)
 				)
@@
 		(dnp no)
 		(fields_autoplaced yes)
-		(property "Reference" "#PWR024"
+		(property "Reference" "#PWR019"
 			(at 102.87 115.57 0)
 			(effects
@@
 			(project "bus"
 				(path "/37ae8b13-e183-404e-b70a-681e1af60f55/61b8f38e-6730-4fc5-8ab9-627730f56fd6"
-					(reference "#PWR024")
+					(reference "#PWR019")
 					(unit 1)
 				)

Commit message: Fixed mismatched RAM labels
Connections:
- net ~{RO} renamed ~{WO}
Changed lines of the file:
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@@
 		)
 	)
-	(hierarchical_label "~{RO}"
+	(hierarchical_label "~{WO}"
 		(shape input)
 		(at 100.33 142.24 180)
