File: Bus/control.kicad_sch (KiCad schematic)
At the start: 3 parts, among them J12 Conn_01x07_Pin, J13 Conn_01x08_Pin, J14 Conn_01x08_Pin

Commit message: Output enable should be active low so I updated control to pass it through an inverter
Connections:
- net Output_EN renamed Output_~{EN}
Changed lines of the file:
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@@
 		)
 	)
-	(hierarchical_label "Output_EN"
+	(hierarchical_label "Output_~{EN}"
 		(shape output)
 		(at 199.39 115.57 180)

Commit message: Bus fully routed. Minor edits to control to match bus
Connections:
- net AR_~{READ}: now also J14.3 (Pin_3); no longer J14.2 (Pin_2)
- net AR_~{WRITE}: now also J14.2 (Pin_2); no longer J14.3 (Pin_3)
- net IR_~{READ}: now also J13.2 (Pin_2); no longer J13.4 (Pin_4)
- net IR_~{WRITE}: now also J13.1 (Pin_1); no longer J13.3 (Pin_3)
- net PC_~{CO}: now also J14.1 (Pin_1); no longer J13.7 (Pin_7)
- net PC_~{JMP}: now also J13.7 (Pin_7); no longer J14.1 (Pin_1)
- net RAM_READ: now also J13.3 (Pin_3); no longer J13.2 (Pin_2)
- net RAM_~{WRITE}: now also J13.4 (Pin_4); no longer J13.1 (Pin_1)
Changed lines of the file:
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@@
 	(hierarchical_label "PC_~{JMP}"
 		(shape output)
-		(at 199.39 97.79 180)
+		(at 199.39 86.36 180)
 		(fields_autoplaced yes)
 		(effects
@@
 	(hierarchical_label "IR_~{WRITE}"
 		(shape output)
-		(at 199.39 76.2 180)
+		(at 199.39 71.12 180)
 		(fields_autoplaced yes)
 		(effects
@@
 	(hierarchical_label "RAM_~{WRITE}"
 		(shape output)
-		(at 199.39 71.12 180)
+		(at 199.39 78.74 180)
 		(fields_autoplaced yes)
 		(effects
@@
 	(hierarchical_label "AR_~{WRITE}"
 		(shape output)
-		(at 199.39 102.87 180)
+		(at 199.39 100.33 180)
 		(fields_autoplaced yes)
 		(effects
@@
 	(hierarchical_label "RAM_READ"
 		(shape output)
+		(at 199.39 76.2 180)
+		(fields_autoplaced yes)
+		(effects
+			(font
+				(size 1.27 1.27)
+			)
+			(justify right)
+		)
+	)
+	(hierarchical_label "BR_~{READ}"
+		(shape output)
+		(at 199.39 113.03 180)
+		(fields_autoplaced yes)
+		(effects
+			(font
+				(size 1.27 1.27)
+			)
+			(justify right)
+		)
+	)
+	(hierarchical_label "RST"
+		(shape output)
+		(at 199.39 64.77 180)
+		(fields_autoplaced yes)
+		(effects
+			(font
+				(size 1.27 1.27)
+			)
+			(justify right)
+		)
+	)
+	(hierarchical_label "MAR_~{EN}"
+		(shape output)
+		(at 199.39 81.28 180)
+		(fields_autoplaced yes)
+		(effects
+			(font
+				(size 1.27 1.27)
+			)
+			(justify right)
+		)
+	)
+	(hierarchical_label "IR_~{READ}"
+		(shape output)
 		(at 199.39 73.66 180)
 		(fields_autoplaced yes)
@@
 		)
 	)
-	(hierarchical_label "BR_~{READ}"
-		(shape output)
-		(at 199.39 113.03 180)
-		(fields_autoplaced yes)
-		(effects
-			(font
-				(size 1.27 1.27)
-			)
-			(justify right)
-		)
-	)
-	(hierarchical_label "RST"
-		(shape output)
-		(at 199.39 64.77 180)
-		(fields_autoplaced yes)
-		(effects
-			(font
-				(size 1.27 1.27)
-			)
-			(justify right)
-		)
-	)
-	(hierarchical_label "MAR_~{EN}"
-		(shape output)
-		(at 199.39 81.28 180)
-		(fields_autoplaced yes)
-		(effects
-			(font
-				(size 1.27 1.27)
-			)
-			(justify right)
-		)
-	)
-	(hierarchical_label "IR_~{READ}"
-		(shape output)
-		(at 199.39 78.74 180)
-		(fields_autoplaced yes)
-		(effects
-			(font
-				(size 1.27 1.27)
-			)
-			(justify right)
-		)
-	)
 	(hierarchical_label "Output_~{EN}"
 		(shape output)
@@
 	(hierarchical_label "PC_~{CO}"
 		(shape output)
-		(at 199.39 86.36 180)
+		(at 199.39 97.79 180)
 		(fields_autoplaced yes)
 		(effects
@@
 	(hierarchical_label "AR_~{READ}"
 		(shape output)
-		(at 199.39 100.33 180)
-		(fields_autoplaced yes)
-		(effects
+		(at 199.39 102.87 180)
+		(fields_autoplaced yes)
+		(effects
