File: RAM/atmega_ram_emulator.kicad_sch (KiCad schematic)
At the start: 6 parts, among them U7 ATMEGA328-PU, Y1 16MHz

Commit message: Fixed incorrect MUX inputs on RAM
Parts:
- renumbered R10 to R18
Changed lines of the file:
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@@
 		(dnp no)
 		(fields_autoplaced yes)
-		(property "Reference" "#PWR026"
+		(property "Reference" "#PWR027"
 			(at 64.77 92.71 0)
 			(effects
@@
 			(project ""
 				(path "/5d332551-33f6-4491-a826-882274bc7f5d/acc97a6d-2734-4118-b9c0-fcc1a4fca6ae"
-					(reference "#PWR026")
-					(unit 1)
-				)
-				(path "/5d332551-33f6-4491-a826-882274bc7f5d/d4879710-3e51-4f6c-bd90-581859fa44c4"
-					(reference "#PWR030")
+					(reference "#PWR027")
+					(unit 1)
+				)
+				(path "/5d332551-33f6-4491-a826-882274bc7f5d/d4879710-3e51-4f6c-bd90-581859fa44c4"
+					(reference "#PWR031")
 					(unit 1)
 				)
@@
 		(dnp no)
 		(fields_autoplaced yes)
-		(property "Reference" "#PWR024"
+		(property "Reference" "#PWR025"
 			(at 38.1 44.45 0)
 			(effects
@@
 			(project "RAM"
 				(path "/5d332551-33f6-4491-a826-882274bc7f5d/acc97a6d-2734-4118-b9c0-fcc1a4fca6ae"
-					(reference "#PWR024")
-					(unit 1)
-				)
-				(path "/5d332551-33f6-4491-a826-882274bc7f5d/d4879710-3e51-4f6c-bd90-581859fa44c4"
-					(reference "#PWR028")
+					(reference "#PWR025")
+					(unit 1)
+				)
+				(path "/5d332551-33f6-4491-a826-882274bc7f5d/d4879710-3e51-4f6c-bd90-581859fa44c4"
+					(reference "#PWR029")
 					(unit 1)
 				)
@@
 		(dnp no)
 		(fields_autoplaced yes)
-		(property "Reference" "#PWR025"
+		(property "Reference" "#PWR026"
 			(at 57.15 30.48 0)
 			(effects
@@
 			(project ""
 				(path "/5d332551-33f6-4491-a826-882274bc7f5d/acc97a6d-2734-4118-b9c0-fcc1a4fca6ae"
-					(reference "#PWR025")
-					(unit 1)
-				)
-				(path "/5d332551-33f6-4491-a826-882274bc7f5d/d4879710-3e51-4f6c-bd90-581859fa44c4"
-					(reference "#PWR029")
+					(reference "#PWR026")
+					(unit 1)
+				)
+				(path "/5d332551-33f6-4491-a826-882274bc7f5d/d4879710-3e51-4f6c-bd90-581859fa44c4"
+					(reference "#PWR030")
 					(unit 1)
 				)
@@
 		(dnp no)
 		(fields_autoplaced yes)
-		(property "Reference" "R10"
+		(property "Reference" "R18"
 			(at 50.8 31.7499 0)
 			(effects
@@
 			(project ""
 				(path "/5d332551-33f6-4491-a826-882274bc7f5d/acc97a6d-2734-4118-b9c0-fcc1a4fca6ae"
-					(reference "R10")
-					(unit 1)
-				)
-				(path "/5d332551-33f6-4491-a826-882274bc7f5d/d4879710-3e51-4f6c-bd90-581859fa44c4"
-					(reference "R11")
+					(reference "R18")
+					(unit 1)
+				)
+				(path "/5d332551-33f6-4491-a826-882274bc7f5d/d4879710-3e51-4f6c-bd90-581859fa44c4"
+					(reference "R19")
 					(unit 1)
 				)
@@
 		(dnp no)
 		(fields_autoplaced yes)
-		(property "Reference" "#PWR027"
+		(property "Reference" "#PWR028"
 			(at 96.52 87.63 0)
 			(effects
@@
 			(project ""
 				(path "/5d332551-33f6-4491-a826-882274bc7f5d/acc97a6d-2734-4118-b9c0-fcc1a4fca6ae"
-					(reference "#PWR027")
-					(unit 1)
-				)
-				(path "/5d332551-33f6-4491-a826-882274bc7f5d/d4879710-3e51-4f6c-bd90-581859fa44c4"
-					(reference "#PWR031")
-					(unit 1)
-				)
+					(reference "#PWR028")
+					(unit 1)
+				)
+				(path "/5d332551-33f6-4491-a826-882274bc7f5d/d4879710-3e51-4f6c-bd90-581859fa44c4"
+					(reference "#PWR032")
+					(unit 1)
+				)
