File: ALU/ALU.kicad_pcb (KiCad board)
At the start: 2 copper layers, 115 x 57 mm, 33 parts, among them J1 Conn_01x06_Pin, J2 Conn_01x08_Pin, J3 Conn_01x08_Pin, J4 Conn_01x10_Pin, U1 SN74F86N, U2 SN74F86N, U3 SN74HCT245N, U4 CD74HCT283E, U5 CD74HCT283E, U8 Dual D FF

Commit message: ALU layout complete
ALU layout complete
Parts:
- added REF**: MountingHole_2.2mm_M2, MountingHole:MountingHole_2.2mm_M2, F.Cu at (78.6, 134.0)
- added REF**: MountingHole_2.2mm_M2, MountingHole:MountingHole_2.2mm_M2, F.Cu at (173.0, 134.0)
- added REF**: MountingHole_2.2mm_M2, MountingHole:MountingHole_2.2mm_M2, F.Cu at (78.6, 85.4)
- added REF**: MountingHole_2.2mm_M2, MountingHole:MountingHole_2.2mm_M2, F.Cu at (173.0, 85.4)
- moved C1 5.06 mm to (87.8, 86.6), turned to 0 degrees
- moved J2 2.91 mm to (98.8, 86.6)
- moved J3 2.26 mm to (98.8, 132.2)
- moved R10 1.80 mm to (162.2, 130.0)
- moved R9 1.69 mm to (148.6, 130.0)
- moved J1 1.20 mm to (78.8, 116.5)
- moved J4 1.20 mm to (78.8, 90.0)
- renumbered D9 to CARRY, D10 to ZERO
Routing:
- net /~{RST}: track 115.9 -> 119.4 mm
- net /CLK: track 115.3 -> 118.4 mm
- net /CARRY: track 97.1 -> 100.2 mm
- net /ZERO: track 103.9 -> 107.0 mm
- net /A6: track 12.0 -> 14.9 mm
- net /A7: track 9.59 -> 12.4 mm
- net /A5: track 26.5 -> 29.3 mm
- net /A4: track 31.3 -> 34.1 mm
- net /XOR0: track 23.0 -> 25.8 mm
- net /A3: track 33.8 -> 36.2 mm
- net /A2: track 27.1 -> 29.6 mm
- net /A0: track 36.1 -> 38.6 mm
- net /B2: track 14.7 -> 17.2 mm
- net /B3: track 12.6 -> 15.0 mm
- net /A1: track 30.5 -> 32.9 mm
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Other:
- board size 115 x 57 mm -> 100.4 x 54.6 mm
- board text added: "0"
- board text added: "1"
- board text added: "2"
- board text added: "2's Complement Inverter"
- board text added: "2x D Flip-Flop"
- board text added: "3"
- board text added: "4"
- board text added: "4-bit Full Adder"
- board text added: "4x AND"
- board text added: "4x NOR"
- board text added: "4x XOR"
- board text added: "5"
- board text added: "6"
- board text added: "7"
- board text added: "8-bit Adder"
- board text added: "8-bit Bus Transciever"
- board text added: "A Register"
- board text added: "ALU"
- board text added: "ALU Flags"
- board text added: "B Register"
- board text added: "B0"
- board text added: "B1"
- board text added: "B2"
- board text added: "B3"
- board text added: "B4"
- board text added: "B5"
- board text added: "B6"
- board text added: "B7"
- board text added: "CLK"
- board text added: "Carry"
- board text added: "GND"
- board text added: "Sub"
- board text added: "VCC"
- board text added: "Zero"
- board text added: "~{RST}"
- board text added: "~{Write}"

Commit message: Fixed misrouted bus connections to MUX. MUX is inverting so adde inverterto invert back. Slide switch should be conencted to power and pulled to ground. Breadboard validated.
Changed lines of the file:
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@@
-	)
-	(gr_arc
-		(start 78.599999 137)
-		(mid 76.478679 136.12132)
-		(end 75.599999 134)
-		(stroke
-			(width 0.05)
-			(type default)
-		)
-		(layer "Edge.Cuts")
 	)
 	(gr_arc
@@
 		(stroke
 			(width 0.05)
+			(type default)
+		)
+		(layer "Edge.Cuts")
+	)
+	(gr_arc
+		(start 78.599998 137)
+		(mid 76.478678 136.12132)
+		(end 75.599998 134)
+		(stroke
+			(width 0.05)

Commit message: Forgot Flags register input enable. Passing clock though spare AND gate with new input Flag In input to create equvilant
Parts:
- J1: value Conn_01x06_Pin -> Conn_01x07_Pin; footprint Connector_PinHeader_2.54mm:PinHeader_1x06_P2.54mm_Vertical -> Connector_PinHeader_2.54mm:PinHeader_1x07_P2.54mm_Vertical
- moved R9 11.6 mm to (160.2, 130.0), turned to 180 degrees
- moved J1 1.28 mm to (78.8, 115.2)
- moved J4 1.25 mm to (78.8, 88.8)
- moved REF** 1.15 mm to (173.0, 84.2)
- moved REF** 1.15 mm to (78.6, 84.2)
- moved REF** 1.00 mm to (78.6, 135.0)
- moved REF** 1.00 mm to (173.0, 135.0)
- renumbered ZERO to D10, CARRY to D9
Connections:
- J1 pad 5: /CARRY -> /Flag enable
- J1 pad 6: /ZERO -> /CARRY
- U6 pad 1: unconnected-(U6-1A-Pad1) -> Net-(U6-1A)
- U6 pad 10: Net-(U6-3B) -> /CLK
- U6 pad 11: Net-(U6-3B) -> /FlagsRegister/all_zero
- U6 pad 12: Net-(U6-4A) -> Net-(U6-2Y)
- U6 pad 13: Net-(U6-4B) -> Net-(U6-1Y)
- U6 pad 2: unconnected-(U6-1B-Pad2) -> Net-(U6-1B)
- U6 pad 3: unconnected-(U6-1Y-Pad3) -> Net-(U6-1Y)
- U6 pad 8: /FlagsRegister/all_zero -> /FlagsRegister/CLK_Gate
- U6 pad 9: Net-(U6-2Y) -> /Flag enable
- U7 pad 1: Net-(U6-2B) -> Net-(U6-1B)
- U7 pad 10: Net-(U6-4B) -> Net-(U6-2A)
- U7 pad 13: Net-(U6-4A) -> Net-(U6-2B)
- U7 pad 4: Net-(U6-2A) -> Net-(U6-1A)
- U8 pad 11: /CLK -> /FlagsRegister/CLK_Gate
- U8 pad 3: /CLK -> /FlagsRegister/CLK_Gate
Routing:
- net /Flag enable: track 0.00 -> 98.2 mm
- net Net-(U6-4B): track 38.3 -> 0.00 mm
- net Net-(U6-4A): track 28.5 -> 0.00 mm
- net Net-(U6-1A): track 0.00 -> 26.2 mm
- net /FlagsRegister/CLK_Gate: track 0.00 -> 20.2 mm
- net Net-(U6-1B): track 0.00 -> 17.4 mm
- net /CLK: track 118.4 -> 101.1 mm
- net Net-(U6-2A): track 18.7 -> 28.3 mm
- net Net-(U6-1Y): track 0.00 -> 9.05 mm
- net +5V: track 59.7 -> 51.0 mm
- net Net-(U6-2B): track 10.7 -> 19.2 mm
- net Net-(D9-K): track 12.4 -> 5.37 mm
- net /FlagsRegister/all_zero: track 16.9 -> 12.0 mm
- net Net-(U6-2Y): track 8.00 -> 11.2 mm
- net /~{RST}: track 119.4 -> 122.2 mm
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Other:
- board size 100.4 x 54.6 mm -> 100.4 x 56.8 mm
- board text added: "FI"
