File: Output/7_segment_shift_register.kicad_sch (KiCad schematic)
At the start: 2 parts, among them U3 74HC595, U6 HDSP-7403

Commit message: Updated output to use 2 4-bit registers instead of 1 8-bit because that's what I have. No longer need the AND for clk enable as registers have an enable pin. Enable is now active low. Reset is now active high
Parts:
- renumbered U6 to U10, U3 to U9
Changed lines of the file:
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@@
 		(dnp no)
 		(fields_autoplaced yes)
-		(property "Reference" "#PWR012"
+		(property "Reference" "#PWR020"
 			(at 92.71 109.22 0)
 			(effects
@@
 			(project "Output"
 				(path "/02a99fb8-2048-4cc8-b7aa-813268289b08/ac84326f-8e35-4922-ad5d-170f017a2aed/1de1b698-6f11-42ef-b753-7cf62e46ba17"
-					(reference "#PWR018")
+					(reference "#PWR020")
 					(unit 1)
 				)
 				(path "/02a99fb8-2048-4cc8-b7aa-813268289b08/ac84326f-8e35-4922-ad5d-170f017a2aed/4ca4684f-5943-401f-ba32-bc7fd1806244"
-					(reference "#PWR015")
+					(reference "#PWR017")
 					(unit 1)
 				)
 				(path "/02a99fb8-2048-4cc8-b7aa-813268289b08/ac84326f-8e35-4922-ad5d-170f017a2aed/829bbd52-3ad2-4fd6-a907-3ff9ff187d62"
-					(reference "#PWR09")
+					(reference "#PWR011")
 					(unit 1)
 				)
 				(path "/02a99fb8-2048-4cc8-b7aa-813268289b08/ac84326f-8e35-4922-ad5d-170f017a2aed/f74b3d93-1b03-45c1-a730-4f8a86419698"
-					(reference "#PWR012")
+					(reference "#PWR014")
 					(unit 1)
 				)
@@
 		(dnp no)
 		(fields_autoplaced yes)
-		(property "Reference" "U3"
+		(property "Reference" "U9"
 			(at 94.9041 104.14 0)
 			(effects
@@
 		(dnp no)
 		(fields_autoplaced yes)
-		(property "Reference" "#PWR010"
+		(property "Reference" "#PWR021"
 			(at 92.71 148.59 0)
 			(effects
@@
 			(project "Output"
 				(path "/02a99fb8-2048-4cc8-b7aa-813268289b08/ac84326f-8e35-4922-ad5d-170f017a2aed/1de1b698-6f11-42ef-b753-7cf62e46ba17"
-					(reference "#PWR019")
+					(reference "#PWR021")
 					(unit 1)
 				)
 				(path "/02a99fb8-2048-4cc8-b7aa-813268289b08/ac84326f-8e35-4922-ad5d-170f017a2aed/4ca4684f-5943-401f-ba32-bc7fd1806244"
-					(reference "#PWR016")
+					(reference "#PWR018")
 					(unit 1)
 				)
 				(path "/02a99fb8-2048-4cc8-b7aa-813268289b08/ac84326f-8e35-4922-ad5d-170f017a2aed/829bbd52-3ad2-4fd6-a907-3ff9ff187d62"
-					(reference "#PWR010")
+					(reference "#PWR012")
 					(unit 1)
 				)
 				(path "/02a99fb8-2048-4cc8-b7aa-813268289b08/ac84326f-8e35-4922-ad5d-170f017a2aed/f74b3d93-1b03-45c1-a730-4f8a86419698"
-					(reference "#PWR013")
+					(reference "#PWR015")
 					(unit 1)
 				)
@@
 		(dnp no)
 		(fields_autoplaced yes)
-		(property "Reference" "U6"
+		(property "Reference" "U10"
 			(at 115.57 101.6 0)
 			(effects
@@
 		(dnp no)
 		(fields_autoplaced yes)
-		(property "Reference" "#PWR014"
+		(property "Reference" "#PWR022"
 			(at 124.46 137.16 0)
 			(effects
@@
 			(project "Output"
 				(path "/02a99fb8-2048-4cc8-b7aa-813268289b08/ac84326f-8e35-4922-ad5d-170f017a2aed/1de1b698-6f11-42ef-b753-7cf62e46ba17"
-					(reference "#PWR020")
+					(reference "#PWR022")
 					(unit 1)
 				)
 				(path "/02a99fb8-2048-4cc8-b7aa-813268289b08/ac84326f-8e35-4922-ad5d-170f017a2aed/4ca4684f-5943-401f-ba32-bc7fd1806244"
-					(reference "#PWR017")
+					(reference "#PWR019")
 					(unit 1)
 				)
 				(path "/02a99fb8-2048-4cc8-b7aa-813268289b08/ac84326f-8e35-4922-ad5d-170f017a2aed/829bbd52-3ad2-4fd6-a907-3ff9ff187d62"
-					(reference "#PWR011")
+					(reference "#PWR013")
 					(unit 1)
 				)
 				(path "/02a99fb8-2048-4cc8-b7aa-813268289b08/ac84326f-8e35-4922-ad5d-170f017a2aed/f74b3d93-1b03-45c1-a730-4f8a86419698"
-					(reference "#PWR014")
-					(unit 1)
-				)
+					(reference "#PWR016")
+					(unit 1)
+				)
