File: Output/Output.kicad_pcb (KiCad board)
At the start: 2 copper layers, 109.7 x 49.5 mm, 18 parts, among them J1 Conn_01x10_Pin, J2 Conn_01x04_Pin, U1 74LS173, U2 74LS173, U3 AT28C64B-15PI, U4 CC56-12CGKWA, U5 NE555P, U6 CD74HCT139E, U7 CD74HCT73E

Commit message: Ouput bus was labeled incorectly. Labels fixed on output. Labels and connections fixed on bus
Changed lines of the file:
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@@
 	)
 	(gr_text "B2"
-		(at 91.948 89.886 0)
+		(at 92.202 82.58 0)
 		(layer "F.SilkS")
 		(effects
@@
 	)
 	(gr_text "B3"
-		(at 91.948 87.386 0)
+		(at 92.202 85.08 0)
 		(layer "F.SilkS")
 		(effects
@@
 	)
 	(gr_text "B4"
-		(at 91.948 84.886 0)
+		(at 92.202 87.58 0)
 		(layer "F.SilkS")
 		(effects
@@
 	)
 	(gr_text "B6"
-		(at 91.948 79.886 0)
+		(at 92.202 92.58 0)
 		(layer "F.SilkS")
 		(effects
@@
 	)
 	(gr_text "B0"
-		(at 91.944 94.996 0)
+		(at 92.198 77.47 0)
 		(layer "F.SilkS")
 		(effects
@@
 	)
 	(gr_text "B1"
-		(at 91.948 92.386 0)
+		(at 92.202 80.08 0)
 		(layer "F.SilkS")
 		(effects
@@
 	)
 	(gr_text "B7"
-		(at 91.948 77.386 0)
+		(at 92.202 95.08 0)
 		(layer "F.SilkS")
 		(effects
@@
 	)
 	(gr_text "B5"
-		(at 91.948 82.386 0)
+		(at 92.202 90.08 0)
 		(layer "F.SilkS")
 		(effects

Commit message: Demux enable is active low. Should have been connected to ground not power
Connections:
- U6 pad 1: +5V -> GND
Changed lines of the file:
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@@
 			(layers "*.Cu" "*.Mask")
 			(remove_unused_layers no)
-			(net 2 "+5V")
+			(net 1 "GND")
 			(pinfunction "*1E")
 			(pintype "input")

Commit message: Added pulling resistors to unused pins from bus. (Output 2s comp & B reg write out)
Parts:
- added R3: 1k, _DownloadFootprints:CF_series_Resistors_THT, F.Cu at (100.8, 78.5)
Routing:
- net /2's Comp: track 46.6 -> 55.0 mm
