File: Output/Output.kicad_sch (KiCad schematic)
At the start: 7 parts, among them J1 Conn_01x10_Pin, J2 Conn_01x04_Pin, U1 74LS173, U2 74LS173, U3 AT28C64B-15PI, U4 CC56-12CGKWA

Commit message: Added pulling resistors to unused pins from bus. (Output 2s comp & B reg write out)
Parts:
- added R3: 1k, _DownloadFootprints:CF_series_Resistors_THT, symbol Device:R
Connections:
- net 2's Comp: now also R3.2
- net GND: now also R3.1
Changed lines of the file:
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@@
 		)
 	)
-	(label "Bus 4"
-		(at 82.55 99.06 180)
+	(label "2's Comp"
+		(at 41.91 78.74 0)
 		(fields_autoplaced yes)
 		(effects
@@
 				(size 1.27 1.27)
 			)
-			(justify right bottom)
-		)
-	)
-	(label "RST"
-		(at 82.55 121.92 180)
+			(justify left bottom)
+		)
+	)
+	(label "Bus 4"
+		(at 82.55 99.06 180)
 		(fields_autoplaced yes)
 		(effects
@@
 		)
 	)
-	(label "g"
-		(at 218.44 100.33 0)
+	(label "RST"
+		(at 82.55 121.92 180)
 		(fields_autoplaced yes)
 		(effects
@@
 				(size 1.27 1.27)
 			)
-			(justify left bottom)
-		)
-	)
-	(label "D0"
-		(at 107.95 40.64 0)
+			(justify right bottom)
+		)
+	)
+	(label "g"
+		(at 218.44 100.33 0)
 		(fields_autoplaced yes)
 		(effects
@@
 		)
 	)
-	(label "Bus 0"
-		(at 82.55 40.64 180)
+	(label "D0"
+		(at 107.95 40.64 0)
 		(fields_autoplaced yes)
 		(effects
@@
 				(size 1.27 1.27)
 			)
-			(justify right bottom)
-		)
-	)
-	(label "DT2"
-		(at 214.63 146.05 0)
+			(justify left bottom)
+		)
+	)
+	(label "Bus 0"
+		(at 82.55 40.64 180)
 		(fields_autoplaced yes)
 		(effects
@@
 				(size 1.27 1.27)
 			)
+			(justify right bottom)
+		)
+	)
+	(label "DT2"
+		(at 214.63 146.05 0)
+		(fields_autoplaced yes)
+		(effects
+			(font
+				(size 1.27 1.27)
+			)
 			(justify left bottom)
 		)
@@
 	)
 	(symbol
+		(lib_id "Device:R")
+		(at 41.91 82.55 0)
+		(mirror x)
+		(unit 1)
+		(exclude_from_sim no)
+		(in_bom yes)
+		(on_board yes)
+		(dnp no)
+		(fields_autoplaced yes)
+		(property "Reference" "R3"
+			(at 39.37 81.2799 0)
+			(effects
+				(font
+					(size 1.27 1.27)
+				)
+				(justify right)
+			)
+		)
+		(property "Value" "1k"
+			(at 39.37 83.8199 0)
+			(effects
+				(font
+					(size 1.27 1.27)
+				)
+				(justify right)
+			)
+		)
+		(property "Footprint" "_DownloadFootprints:CF_series_Resistors_THT"
+			(at 40.132 82.55 90)
+			(effects
+				(font
+					(size 1.27 1.27)
+				)
+				(hide yes)
+			)
+		)
+		(property "Datasheet" "~"
+			(at 41.91 82.55 0)
+			(effects
+				(font
+					(size 1.27 1.27)
+				)
+				(hide yes)
+			)
+		)
+		(property "Description" "Resistor"
+			(at 41.91 82.55 0)
+			(effects
+				(font
+					(size 1.27 1.27)
+				)
+				(hide yes)
+			)
+		)
+		(pin "2"
+		)
+		(pin "1"
+		)
+		(instances
+			(project "Output"
+				(path "/02a99fb8-2048-4cc8-b7aa-813268289b08"
+					(reference "R3")
+					(unit 1)
+				)
+			)
+		)
+	)
+	(symbol
 		(lib_id "eeprom:AT28C64B-15PI")
 		(at 157.48 69.85 0)
@@
 					(unit 1)
 				)
+			)
+		)
+	)
+	(symbol
+		(lib_id "power:GND")
+		(at 41.91 86.36 0)
+		(unit 1)
+		(exclude_from_sim no)
+		(in_bom yes)
+		(on_board yes)
+		(dnp no)
+		(fields_autoplaced yes)
+		(property "Reference" "#PWR024"
+			(at 41.91 92.71 0)
+			(effects
+				(font
+					(size 1.27 1.27)
+				)
+				(hide yes)
+			)
+		)
+		(property "Value" "GND"
+			(at 41.91 91.44 0)
+			(effects
+				(font
+					(size 1.27 1.27)
+				)
+			)
+		)
+		(property "Footprint" ""
+			(at 41.91 86.36 0)
+			(effects
+				(font
+					(size 1.27 1.27)
+				)
+				(hide yes)
+			)
+		)
+		(property "Datasheet" ""
+			(at 41.91 86.36 0)
+			(effects
+				(font
+					(size 1.27 1.27)
+				)
+				(hide yes)
+			)
+		)
+		(property "Description" "Power symbol creates a global label with name \"GND\" , ground"
+			(at 41.91 86.36 0)
+			(effects
+				(font
+					(size 1.27 1.27)
+				)
+				(hide yes)
+			)
+		)
+		(pin "1"
+		)
+		(instances
+			(project ""
+				(path "/02a99fb8-2048-4cc8-b7aa-813268289b08"
+					(reference "#PWR024")
+					(unit 1)
+				)
