File: Control/Control.kicad_sch (KiCad schematic)
At the start: 13 parts, among them J1 Conn_01x03_Pin, J2 Conn_01x04_Pin, J3 Conn_01x08_Pin, J4 Conn_01x08_Pin, J5 Conn_01x07_Pin, U1 AT28C64B-15PI, U2 AT28C64B-15PI, U3 SN74AC14N, U4 SN74AC14N

Commit message: Bus fully routed. Minor edits to control to match bus
Connections:
- net AR_RI: now also U1.18 (I/O6), U3.13 (6A); no longer U1.19 (I/O7), U3.11 (5A)
- net AR_WO: now also U1.19 (I/O7), U3.11 (5A); no longer U1.18 (I/O6), U3.13 (6A)
- net IR_RI: now also U2.16 (I/O4), U4.11 (5A); no longer U2.18 (I/O6), U4.1 (1A)
- net IR_WO: now also U2.15 (I/O3), U4.13 (6A); no longer U2.16 (I/O4), U4.11 (5A)
- net PC_CO: now also U1.11 (I/O0), U3.9 (4A); no longer U1.15 (I/O3), U4.5 (3A)
- net PC_JMP: now also U1.15 (I/O3), U4.5 (3A); no longer U1.11 (I/O0), U3.9 (4A)
- net RAM_RI: now also J3.3 (Pin_3); no longer J3.2 (Pin_2)
- net RAM_WO: now also U2.18 (I/O6), U4.1 (1A); no longer U2.15 (I/O3), U4.13 (6A)
- net ~{AR_RI}: now also J4.3 (Pin_3), U3.12 (6Y); no longer J4.2 (Pin_2), U3.10 (5Y)
- net ~{AR_WO}: now also J4.2 (Pin_2), U3.10 (5Y); no longer J4.3 (Pin_3), U3.12 (6Y)
- net ~{IR_RI}: now also J3.2 (Pin_2), U4.10 (5Y); no longer J3.4 (Pin_4), U4.2 (1Y)
- net ~{IR_WO}: now also J3.1 (Pin_1), U4.12 (6Y); no longer J3.3 (Pin_3), U4.10 (5Y)
- net ~{PC_CO}: now also J4.1 (Pin_1), U3.8 (4Y); no longer J3.7 (Pin_7), U4.6 (3Y)
- net ~{PC_JMP}: now also J3.7 (Pin_7), U4.6 (3Y); no longer J4.1 (Pin_1), U3.8 (4Y)
- net ~{RAM_WO}: now also J3.4 (Pin_4), U4.2 (1Y); no longer J3.1 (Pin_1), U4.12 (6Y)
Changed lines of the file:
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@@
 	)
 	(label "~{RAM_WO}"
-		(at 226.06 83.82 0)
-		(fields_autoplaced yes)
-		(effects
-			(font
-				(size 1.27 1.27)
-			)
-			(justify left bottom)
+		(at 170.18 81.28 180)
+		(fields_autoplaced yes)
+		(effects
+			(font
+				(size 1.27 1.27)
+			)
+			(justify right bottom)
 		)
 	)
@@
 	)
 	(label "PC_JMP"
-		(at 226.06 59.69 0)
-		(fields_autoplaced yes)
-		(effects
-			(font
-				(size 1.27 1.27)
-			)
-			(justify left bottom)
+		(at 170.18 88.9 180)
+		(fields_autoplaced yes)
+		(effects
+			(font
+				(size 1.27 1.27)
+			)
+			(justify right bottom)
 		)
 	)
@@
 	)
 	(label "~{IR_WO}"
-		(at 261.62 36.83 180)
+		(at 261.62 31.75 180)
 		(fields_autoplaced yes)
 		(effects
@@
 	)
 	(label "IR_WO"
-		(at 226.06 86.36 0)
+		(at 226.06 81.28 0)
 		(fields_autoplaced yes)
 		(effects
@@
 	)
 	(label "IR_WO"
-		(at 100.33 113.03 0)
+		(at 100.33 115.57 0)
 		(fields_autoplaced yes)
 		(effects
@@
 	)
 	(label "RAM_WO"
-		(at 100.33 115.57 0)
+		(at 100.33 107.95 0)
 		(fields_autoplaced yes)
 		(effects
@@
 	)
 	(label "PC_CO"
-		(at 170.18 88.9 180)
-		(fields_autoplaced yes)
-		(effects
-			(font
-				(size 1.27 1.27)
-			)
-			(justify right bottom)
+		(at 226.06 59.69 0)
+		(fields_autoplaced yes)
+		(effects
+			(font
+				(size 1.27 1.27)
+			)
+			(justify left bottom)
 		)
 	)
@@
 	)
 	(label "RAM_RI"
-		(at 261.62 34.29 180)
+		(at 261.62 36.83 180)
 		(fields_autoplaced yes)
 		(effects
@@
 	)
 	(label "AR_WO"
-		(at 100.33 58.42 0)
+		(at 100.33 55.88 0)
 		(fields_autoplaced yes)
 		(effects
@@
 	)
 	(label "~{IR_RI}"
-		(at 170.18 81.28 180)
-		(fields_autoplaced yes)
-		(effects
-			(font
-				(size 1.27 1.27)
-			)
-			(justify right bottom)
+		(at 226.06 88.9 0)
+		(fields_autoplaced yes)
+		(effects
+			(font
+				(size 1.27 1.27)
+			)
+			(justify left bottom)
 		)
 	)
@@
 	)
 	(label "AR_RI"
-		(at 100.33 55.88 0)
+		(at 100.33 58.42 0)
 		(fields_autoplaced yes)
 		(effects
@@
 	)
 	(label "~{PC_CO}"
-		(at 170.18 91.44 180)
-		(fields_autoplaced yes)
-		(effects
-			(font
-				(size 1.27 1.27)
-			)
-			(justify right bottom)
+		(at 226.06 62.23 0)
+		(fields_autoplaced yes)
+		(effects
+			(font
+				(size 1.27 1.27)
+			)
+			(justify left bottom)
 		)
 	)
@@
 	)
 	(label "~{IR_RI}"
-		(at 261.62 39.37 180)
+		(at 261.62 34.29 180)
 		(fields_autoplaced yes)
 		(effects
@@
 	)
 	(label "AR_WO"
-		(at 226.06 49.53 0)
+		(at 226.06 54.61 0)
 		(fields_autoplaced yes)
 		(effects
@@
 	)
 	(label "~{RAM_WO}"
-		(at 261.62 31.75 180)
+		(at 261.62 39.37 180)
 		(fields_autoplaced yes)
 		(effects
@@
 	)
 	(label "RAM_WO"
-		(at 226.06 81.28 0)
-		(fields_autoplaced yes)
-		(effects
-			(font
-				(size 1.27 1.27)
-			)
-			(justify left bottom)
+		(at 170.18 78.74 180)
+		(fields_autoplaced yes)
+		(effects
+			(font
+				(size 1.27 1.27)
+			)
+			(justify right bottom)
 		)
 	)
@@
 	)
 	(label "~{AR_RI}"
+		(at 226.06 52.07 0)
+		(fields_autoplaced yes)
+		(effects
+			(font
+				(size 1.27 1.27)
+			)
+			(justify left bottom)
+		)
+	)
+	(label "~{AR_WO}"
 		(at 226.06 57.15 0)
-		(fields_autoplaced yes)
-		(effects
-			(font
-				(size 1.27 1.27)
-			)
-			(justify left bottom)
-		)
-	)
-	(label "~{AR_WO}"
-		(at 226.06 52.07 0)
 		(fields_autoplaced yes)
 		(effects
@@
 	)
 	(label "~{PC_JMP}"
-		(at 226.06 62.23 0)
-		(fields_autoplaced yes)
-		(effects
-			(font
-				(size 1.27 1.27)
-			)
-			(justify left bottom)
+		(at 170.18 91.44 180)
+		(fields_autoplaced yes)
+		(effects
+			(font
+				(size 1.27 1.27)
+			)
+			(justify right bottom)
 		)
 	)
@@
 	)
 	(label "PC_JMP"
-		(at 39.37 58.42 180)
-		(fields_autoplaced yes)
-		(effects
-			(font
-				(size 1.27 1.27)
-			)
-			(justify right bottom)
+		(at 100.33 66.04 0)
+		(fields_autoplaced yes)
+		(effects
+			(font
+				(size 1.27 1.27)
+			)
+			(justify left bottom)
 		)
 	)
 	(label "~{AR_WO}"
-		(at 261.62 63.5 180)
+		(at 261.62 60.96 180)
 		(fields_autoplaced yes)
 		(effects
@@
 	)
 	(label "~{PC_JMP}"
-		(at 261.62 58.42 180)
+		(at 261.62 46.99 180)
 		(fields_autoplaced yes)
 		(effects
@@
 	)
 	(label "AR_RI"
-		(at 226.06 54.61 0)
+		(at 226.06 49.53 0)
 		(fields_autoplaced yes)
 		(effects
@@
 	)
 	(label "IR_RI"
-		(at 100.33 107.95 0)
+		(at 100.33 113.03 0)
 		(fields_autoplaced yes)
 		(effects
@@
 	)
 	(label "IR_RI"
-		(at 170.18 78.74 180)
-		(fields_autoplaced yes)
-		(effects
-			(font
-				(size 1.27 1.27)
-			)
-			(justify right bottom)
+		(at 226.06 86.36 0)
+		(fields_autoplaced yes)
+		(effects
+			(font
+				(size 1.27 1.27)
+			)
+			(justify left bottom)
 		)
 	)
@@
 	)
 	(label "~{PC_CO}"
-		(at 261.62 46.99 180)
+		(at 261.62 58.42 180)
 		(fields_autoplaced yes)
 		(effects
@@
 	)
 	(label "~{IR_WO}"
-		(at 226.06 88.9 0)
+		(at 226.06 83.82 0)
 		(fields_autoplaced yes)
 		(effects
@@
 	)
 	(label "~{AR_RI}"
-		(at 261.62 60.96 180)
+		(at 261.62 63.5 180)
 		(fields_autoplaced yes)
 		(effects
@@
 	)
 	(label "PC_CO"
-		(at 100.33 66.04 0)
-		(fields_autoplaced yes)
-		(effects
-			(font
-				(size 1.27 1.27)
-			)
-			(justify left bottom)
-		)
-	)
+		(at 39.37 58.42 180)
+		(fields_autoplaced yes)
+		(effects
+			(font
+				(size 1.27 1.27)
+			)
+			(justify right bottom)
+		)
+	)
