File: Control/reset.kicad_sch (KiCad schematic)
At the start: 7 parts, among them SW1 SW_MEC_5E, U7 74HCT00

Commit message: Control routed on PCB
Parts:
- R20, R21, R22, R23, R24: footprint (none) -> _DownloadFootprints:CF_series_Resistors_THT
- SW1: footprint (none) -> _DownloadFootprints:tactile_switch
- U7: footprint (none) -> Package_DIP:DIP-14_W7.62mm
Changed lines of the file:
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@@
 			)
 		)
-		(property "Footprint" ""
+		(property "Footprint" "Package_DIP:DIP-14_W7.62mm"
 			(at 109.22 48.26 0)
 			(effects
@@
 			)
 		)
-		(property "Footprint" ""
+		(property "Footprint" "Package_DIP:DIP-14_W7.62mm"
 			(at 109.22 78.74 0)
 			(effects
@@
 			)
 		)
-		(property "Footprint" ""
+		(property "Footprint" "_DownloadFootprints:CF_series_Resistors_THT"
 			(at 118.872 44.45 90)
 			(effects
@@
 			)
 		)
-		(property "Footprint" ""
+		(property "Footprint" "_DownloadFootprints:tactile_switch"
 			(at 81.28 41.91 0)
 			(effects
@@
 			)
 		)
-		(property "Footprint" ""
+		(property "Footprint" "_DownloadFootprints:CF_series_Resistors_THT"
 			(at 118.872 88.9 90)
 			(effects
@@
 			)
 		)
-		(property "Footprint" ""
+		(property "Footprint" "_DownloadFootprints:CF_series_Resistors_THT"
 			(at 118.872 74.93 90)
 			(effects
@@
 			)
 		)
-		(property "Footprint" ""
+		(property "Footprint" "Package_DIP:DIP-14_W7.62mm"
 			(at 152.4 52.07 0)
 			(effects
@@
 			)
 		)
-		(property "Footprint" ""
+		(property "Footprint" "_DownloadFootprints:CF_series_Resistors_THT"
 			(at 118.872 60.96 90)
 			(effects
@@
 			)
 		)
-		(property "Footprint" ""
+		(property "Footprint" "_DownloadFootprints:CF_series_Resistors_THT"
 			(at 87.122 54.61 90)
 			(effects
@@
 			)
 		)
-		(property "Footprint" ""
+		(property "Footprint" "Package_DIP:DIP-14_W7.62mm"
 			(at 109.22 92.71 0)
 			(effects
@@
 			)
 		)
-		(property "Footprint" ""
+		(property "Footprint" "Package_DIP:DIP-14_W7.62mm"
 			(at 109.22 64.77 0)
 			(effects

Commit message: Updated microcode timer LEDs to 1 hot signal instead of binary counter
Parts:
- renumbered R20 to R22, R21 to R23, R22 to R24, R23 to R25, R24 to R26
Changed lines of the file:
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@@
 		(dnp no)
 		(fields_autoplaced yes)
-		(property "Reference" "R21"
+		(property "Reference" "R23"
 			(at 123.19 43.1799 0)
 			(effects
@@
 			(project "Control"
 				(path "/460bc1d8-5a70-4cad-87d6-3febe61be174/713e61f2-2f45-47e3-a661-3fcccc9dd80f"
-					(reference "R21")
+					(reference "R23")
 					(unit 1)
 				)
@@
 		(dnp no)
 		(fields_autoplaced yes)
-		(property "Reference" "R24"
+		(property "Reference" "R26"
 			(at 123.19 87.6299 0)
 			(effects
@@
 			(project "Control"
 				(path "/460bc1d8-5a70-4cad-87d6-3febe61be174/713e61f2-2f45-47e3-a661-3fcccc9dd80f"
-					(reference "R24")
+					(reference "R26")
 					(unit 1)
 				)
@@
 		(dnp no)
 		(fields_autoplaced yes)
-		(property "Reference" "R23"
+		(property "Reference" "R25"
 			(at 123.19 73.6599 0)
 			(effects
@@
 			(project "Control"
 				(path "/460bc1d8-5a70-4cad-87d6-3febe61be174/713e61f2-2f45-47e3-a661-3fcccc9dd80f"
-					(reference "R23")
+					(reference "R25")
 					(unit 1)
 				)
@@
 		(dnp no)
 		(fields_autoplaced yes)
-		(property "Reference" "R22"
+		(property "Reference" "R24"
 			(at 123.19 59.6899 0)
 			(effects
@@
 			(project "Control"
 				(path "/460bc1d8-5a70-4cad-87d6-3febe61be174/713e61f2-2f45-47e3-a661-3fcccc9dd80f"
-					(reference "R22")
+					(reference "R24")
 					(unit 1)
 				)
@@
 		(dnp no)
 		(fields_autoplaced yes)
-		(property "Reference" "R20"
+		(property "Reference" "R22"
 			(at 91.44 53.3399 0)
 			(effects
@@
 			(project ""
 				(path "/460bc1d8-5a70-4cad-87d6-3febe61be174/713e61f2-2f45-47e3-a661-3fcccc9dd80f"
-					(reference "R20")
-					(unit 1)
-				)
+					(reference "R22")
+					(unit 1)
+				)

Commit message: Added spare pins to control
Parts:
- renumbered R22 to R25, R23 to R26, R24 to R27, R25 to R28, R26 to R29
Changed lines of the file:
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@@
 		(dnp no)
 		(fields_autoplaced yes)
-		(property "Reference" "#PWR034"
+		(property "Reference" "#PWR031"
 			(at 88.9 66.04 0)
 			(effects
@@
 			(project ""
 				(path "/460bc1d8-5a70-4cad-87d6-3febe61be174/713e61f2-2f45-47e3-a661-3fcccc9dd80f"
-					(reference "#PWR034")
+					(reference "#PWR031")
 					(unit 1)
 				)
@@
 		(dnp no)
 		(fields_autoplaced yes)
-		(property "Reference" "#PWR033"
+		(property "Reference" "#PWR030"
 			(at 73.66 49.53 0)
 			(effects
@@
 			(project ""
 				(path "/460bc1d8-5a70-4cad-87d6-3febe61be174/713e61f2-2f45-47e3-a661-3fcccc9dd80f"
-					(reference "#PWR033")
+					(reference "#PWR030")
 					(unit 1)
 				)
@@
 		(dnp no)
 		(fields_autoplaced yes)
-		(property "Reference" "R23"
+		(property "Reference" "R26"
 			(at 123.19 43.1799 0)
 			(effects
@@
 			(project "Control"
 				(path "/460bc1d8-5a70-4cad-87d6-3febe61be174/713e61f2-2f45-47e3-a661-3fcccc9dd80f"
-					(reference "R23")
+					(reference "R26")
 					(unit 1)
 				)
@@
 		(dnp no)
 		(fields_autoplaced yes)
-		(property "Reference" "#PWR039"
+		(property "Reference" "#PWR036"
 			(at 152.4 43.18 0)
 			(effects
@@
 			(project ""
 				(path "/460bc1d8-5a70-4cad-87d6-3febe61be174/713e61f2-2f45-47e3-a661-3fcccc9dd80f"
-					(reference "#PWR039")
+					(reference "#PWR036")
 					(unit 1)
 				)
@@
 		(dnp no)
 		(fields_autoplaced yes)
-		(property "Reference" "#PWR036"
+		(property "Reference" "#PWR033"
 			(at 120.65 60.96 0)
 			(effects
@@
 			(project "Control"
 				(path "/460bc1d8-5a70-4cad-87d6-3febe61be174/713e61f2-2f45-47e3-a661-3fcccc9dd80f"
-					(reference "#PWR036")
+					(reference "#PWR033")
 					(unit 1)
 				)
@@
 		(dnp no)
 		(fields_autoplaced yes)
-		(property "Reference" "#PWR035"
+		(property "Reference" "#PWR032"
 			(at 120.65 44.45 0)
 			(effects
@@
 			(project "Control"
 				(path "/460bc1d8-5a70-4cad-87d6-3febe61be174/713e61f2-2f45-47e3-a661-3fcccc9dd80f"
-					(reference "#PWR035")
+					(reference "#PWR032")
 					(unit 1)
 				)
@@
 		(dnp no)
 		(fields_autoplaced yes)
-		(property "Reference" "#PWR040"
+		(property "Reference" "#PWR037"
 			(at 152.4 71.12 0)
 			(effects
@@
 			(project ""
 				(path "/460bc1d8-5a70-4cad-87d6-3febe61be174/713e61f2-2f45-47e3-a661-3fcccc9dd80f"
-					(reference "#PWR040")
+					(reference "#PWR037")
 					(unit 1)
 				)
@@
 		(dnp no)
 		(fields_autoplaced yes)
-		(property "Reference" "#PWR038"
+		(property "Reference" "#PWR035"
 			(at 120.65 88.9 0)
 			(effects
@@
 			(project "Control"
 				(path "/460bc1d8-5a70-4cad-87d6-3febe61be174/713e61f2-2f45-47e3-a661-3fcccc9dd80f"
-					(reference "#PWR038")
+					(reference "#PWR035")
 					(unit 1)
 				)
@@
 		(dnp no)
 		(fields_autoplaced yes)
-		(property "Reference" "#PWR037"
+		(property "Reference" "#PWR034"
 			(at 120.65 74.93 0)
 			(effects
@@
 			(project "Control"
 				(path "/460bc1d8-5a70-4cad-87d6-3febe61be174/713e61f2-2f45-47e3-a661-3fcccc9dd80f"
-					(reference "#PWR037")
+					(reference "#PWR034")
 					(unit 1)
 				)
@@
 		(dnp no)
 		(fields_autoplaced yes)
-		(property "Reference" "R26"
+		(property "Reference" "R29"
 			(at 123.19 87.6299 0)
 			(effects
@@
 			(project "Control"
 				(path "/460bc1d8-5a70-4cad-87d6-3febe61be174/713e61f2-2f45-47e3-a661-3fcccc9dd80f"
-					(reference "R26")
+					(reference "R29")
 					(unit 1)
 				)
@@
 		(dnp no)
 		(fields_autoplaced yes)
-		(property "Reference" "R25"
+		(property "Reference" "R28"
 			(at 123.19 73.6599 0)
 			(effects
@@
 			(project "Control"
 				(path "/460bc1d8-5a70-4cad-87d6-3febe61be174/713e61f2-2f45-47e3-a661-3fcccc9dd80f"
-					(reference "R25")
+					(reference "R28")
 					(unit 1)
 				)
@@
 		(dnp no)
 		(fields_autoplaced yes)
-		(property "Reference" "R24"
+		(property "Reference" "R27"
 			(at 123.19 59.6899 0)
 			(effects
@@
 			(project "Control"
 				(path "/460bc1d8-5a70-4cad-87d6-3febe61be174/713e61f2-2f45-47e3-a661-3fcccc9dd80f"
-					(reference "R24")
+					(reference "R27")
 					(unit 1)
 				)
@@
 		(dnp no)
 		(fields_autoplaced yes)
-		(property "Reference" "R22"
+		(property "Reference" "R25"
 			(at 91.44 53.3399 0)
 			(effects
@@
 			(project ""
 				(path "/460bc1d8-5a70-4cad-87d6-3febe61be174/713e61f2-2f45-47e3-a661-3fcccc9dd80f"
-					(reference "R22")
-					(unit 1)
-				)
+					(reference "R25")
+					(unit 1)
+				)

Commit message: Control reset signals were inverted
Connections:
- net RST: now also R27.2, U7.6; no longer R26.2, U7.3, U7.4, U7.5, U7.9
- net ~{RST}: now also R26.2, U7.3, U7.4, U7.5, U7.9; no longer R27.2, U7.6
Changed lines of the file:
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@@
 	(hierarchical_label "~{RST}"
 		(shape output)
-		(at 124.46 64.77 0)
+		(at 124.46 48.26 0)
 		(fields_autoplaced yes)
 		(effects
@@
 	(hierarchical_label "RST"
 		(shape output)
-		(at 124.46 48.26 0)
+		(at 124.46 64.77 0)
 		(fields_autoplaced yes)
 		(effects
